File: KiCad/4WireFanController.kicad_sch (KiCad schematic)
At the start: 15 parts, among them M1 Fan_4pin, Q1 BSS214NW, Q2 BSS214NW, SW1 RotaryEncoder_Switch

Commit message: Add files via upload
Parts:
- removed Q2: BSS214NW, Package_TO_SOT_SMD:SOT-323_SC-70, symbol Transistor_FET:BSS214NW
- removed R3: 330, Resistor_SMD:R_0603_1608Metric_Pad0.98x0.95mm_HandSolder, symbol Device:R_US
- removed R4: 100k, Resistor_SMD:R_0603_1608Metric_Pad0.98x0.95mm_HandSolder, symbol Device:R_US
- Q1: footprint Package_TO_SOT_SMD:SOT-323_SC-70 -> Package_TO_SOT_SMD:SOT-23-3
Connections:
- net TACH: now also M1.3 (Tacho)
Other:
- note added: "Step 0 write code to accept serial (USB) text commands parse the commands and output data over serial (USB)"
- moved on the sheet: R5
